Commit message: Gazebo project and improved second project

File: Project 2: Go chase it/my_robot/urdf/my_robot_improved.xacro (robot description, xacro)
@@ -1,5 +1,5 @@
 <?xml version='1.0'?>
 <robot name="my_robot" xmlns:xacro="http://www.ros.org/wiki/xacro">
-  <xacro:include filename="$(find my_robot)/urdf/my_robot.gazebo" />
+  <xacro:include filename="$(find my_robot)/urdf/my_robot_improved.gazebo" />
   <link name="robot_footprint"></link>
   <joint name="robot_footprint_joint" type="fixed">
@@ -9,5 +9,5 @@
   </joint>
   <link name='chassis'>
-    <pose>0 0 0.15 0 0 0</pose>
+    <pose>0 0 0 0 0 0</pose>
     <inertial>
       <mass value="15.0"/>
@@ -22,35 +22,35 @@
       <origin xyz="0 0 0" rpy=" 0 0 0"/>
       <geometry>
-        <box size=".5 .25 .15"/>
+        <box size=".58 .3 .08"/>
       </geometry>
     </collision>
     <visual name='chassis_visual'>
-      <origin xyz="0 0 0" rpy=" 0 0 0"/>
+      <origin xyz="0 0 0" rpy="0 0 0"/>
       <geometry>
-        <box size=".5 .25 .15"/>
+        <mesh filename="package://my_robot/meshes/chassis.dae" scale="1 1 1"/>
       </geometry>
     </visual>
     <collision name='back_caster_collision'>
-      <origin xyz="-0.15 0 -0.075" rpy=" 0 0 0"/>
+      <origin xyz="-0.25 0 0.01" rpy=" 0 0 0"/>
       <geometry>
-        <sphere radius="0.07499"/>
+        <sphere radius="0.0099"/>
       </geometry>
     </collision>
     <visual name='back_caster_visual'>
-      <origin xyz="-0.15 0 -0.075" rpy=" 0 0 0"/>
+      <origin xyz="-0.25 0 0.01" rpy=" 0 0 0"/>
       <geometry>
-        <sphere radius="0.075"/>
+        <sphere radius="0.01"/>
       </geometry>
     </visual>
     <collision name='front_caster_collision'>
-      <origin xyz="0.15 0 -0.075" rpy=" 0 0 0"/>
+      <origin xyz="0.25 0 0.01" rpy=" 0 0 0"/>
       <geometry>
-        <sphere radius="0.07499"/>
+        <sphere radius="0.0099"/>
       </geometry>
     </collision>
     <visual name='front_caster_visual'>
-      <origin xyz="0.15 0 -0.075" rpy=" 0 0 0"/>
+      <origin xyz="0.25 0 0.01" rpy=" 0 0 0"/>
       <geometry>
-        <sphere radius="0.075"/>
+        <sphere radius="0.01"/>
       </geometry>
     </visual>
@@ -58,12 +58,12 @@
   <link name='right_wheel'>
     <visual name='right_wheel_visual'>
-      <origin xyz="0 0 0" rpy="0 1.5707 1.5707"/>
+      <origin xyz="0 0 0" rpy="0 0 0"/>
       <geometry>
-        <cylinder length="0.05" radius="0.15"/>
+        <mesh filename="package://my_robot/meshes/right_wheel.dae" scale="1 1 1"/>
       </geometry>
     </visual>
     <inertial>
       <mass value="5"/>
-      <origin xyz="0 0 0" rpy="0 1.5707 1.5707"/>
+      <origin xyz="0 0 0" rpy="0 0 0"/>
       <inertia
           ixx="0.1" ixy="0" ixz="0"
@@ -73,7 +73,7 @@
     </inertial>
     <collision name='right_wheel_collision'>
-      <origin xyz="0 0 0" rpy="0 1.5707 1.5707"/>
+      <origin xyz="0 0 0" rpy="0 0 0"/>
       <geometry>
-        <cylinder length="0.05" radius="0.15"/>
+        <cylinder length="0.035" radius="0.055"/>
       </geometry>
     </collision>
@@ -81,12 +81,12 @@
   <link name='left_wheel'>
     <visual name='left_wheel_visual'>
-      <origin xyz="0 0 0" rpy="0 1.5707 1.5707"/>
+      <origin xyz="0 0 0" rpy="0 0 0"/>
       <geometry>
-        <cylinder length="0.05" radius="0.15"/>
+        <mesh filename="package://my_robot/meshes/left_wheel.dae" scale="1 1 1"/>
       </geometry>
     </visual>
     <inertial>
       <mass value="5"/>
-      <origin xyz="0 0 0" rpy="0 1.5707 1.5707"/>
+      <origin xyz="0 0 0" rpy="0 0 0"/>
       <inertia
           ixx="0.1" ixy="0" ixz="0"
@@ -96,12 +96,12 @@
     </inertial>
     <collision name='left_wheel_collision'>
-      <origin xyz="0 0 0" rpy="0 1.5707 1.5707"/>
+      <origin xyz="0 0 0" rpy="0 0 0"/>
       <geometry>
-        <cylinder length="0.05" radius="0.15"/>
+        <cylinder length="0.035" radius="0.055"/>
       </geometry>
     </collision>
   </link>
   <joint type="continuous" name="left_wheel_hinge">
-    <origin xyz="0 0.2 0" rpy="0 0 0"/>
+    <origin xyz="-0.17 0.1325 0.055" rpy="0 0 0"/>
     <child link="left_wheel"/>
     <parent link="chassis"/>
@@ -111,5 +111,5 @@
   </joint>
   <joint type="continuous" name="right_wheel_hinge">
-    <origin xyz="0 -0.2 0" rpy="0 0 0"/>
+    <origin xyz="-0.17 -0.1325 0.055" rpy="0 0 0"/>
     <child link="right_wheel"/>
     <parent link="chassis"/>
@@ -122,5 +122,5 @@
       <origin xyz="0 0 0" rpy="0 0 0"/>
       <geometry>
-        <box size=".05 .05 .05"/>
+        <box size=".03 .03 .03"/>
       </geometry>
     </visual>
@@ -137,10 +137,10 @@
       <origin xyz="0 0 0" rpy="0 0 0"/>
       <geometry>
-        <box size=".05 .05 .05"/>
+        <box size=".03 .03 .03"/>
       </geometry>
     </collision>
   </link>
   <joint type="fixed" name="camera_joint">
-    <origin xyz="0.25 0 0" rpy="0 0 0"/>
+    <origin xyz="0.275 0 0.07" rpy="0 0 0"/>
     <child link="camera"/>
     <parent link="chassis"/>
@@ -171,5 +171,5 @@
   </link>
   <joint type="fixed" name="hokuyo_joint">
-    <origin xyz="0.2 0 0.15" rpy="0 0 0"/>
+    <origin xyz="-0.15 0 0.12" rpy="0 0 0"/>
     <child link="hokuyo"/>
     <parent link="chassis"/>
@@ -177,14 +177,14 @@
   </joint>
   <gazebo reference="left_wheel">
-    <material>Gazebo/Black</material>
+    <material>Gazebo/Green</material>
   </gazebo>
   <gazebo reference="right_wheel">
-    <material>Gazebo/Black</material>
+    <material>Gazebo/Green</material>
   </gazebo>
   <gazebo reference="chassis">
+    <material>Gazebo/Blue</material>
+  </gazebo>
+  <gazebo reference="camera">
     <material>Gazebo/Red</material>
   </gazebo>
-  <gazebo reference="camera">
-    <material>Gazebo/Blue</material>
-  </gazebo>
 </robot>
