Commit message: project mapping

File: Project 4: Map my world/my_robot/urdf/udacity_robot.xacro (robot description, xacro)
@@ -59,5 +59,5 @@
     <pose>0 0 0 0 0 0</pose>
     <inertial>
-      <mass value="5.0"/>
+      <mass value="2.0"/>
       <origin xyz="0.0 0.0 0.0" rpy="0 1.5707 1.5707"/>
       <inertia
@@ -83,5 +83,5 @@
     <pose>0 0 0 0 0 0</pose>
     <inertial>
-      <mass value="5.0"/>
+      <mass value="2.0"/>
       <origin xyz="0.0 0.0 0.0" rpy="0 1.5707 1.5707"/>
       <inertia
