Commit message: Mapping project implemented

File: Project 4: Map my world/my_robot/urdf/my_robot.xacro (robot description, xacro)
@@ -11,5 +11,5 @@
     <pose>0 0 0.15 0 0 0</pose>
     <inertial>
-      <mass value="15.0"/>
+      <mass value="4.0"/>
       <origin xyz="0.0 0 0" rpy=" 0 0 0"/>
       <inertia
@@ -64,5 +64,5 @@
     </visual>
     <inertial>
-      <mass value="5"/>
+      <mass value="1.5"/>
       <origin xyz="0 0 0" rpy="0 1.5707 1.5707"/>
       <inertia
@@ -87,5 +87,5 @@
     </visual>
     <inertial>
-      <mass value="5"/>
+      <mass value="1.5"/>
       <origin xyz="0 0 0" rpy="0 1.5707 1.5707"/>
       <inertia

File: Project 4: Map my world/my_robot/urdf/udacity_robot.xacro (robot description, xacro)
@@ -11,5 +11,5 @@
     <pose>0 0 0.1 0 0 0</pose>
     <inertial>
-      <mass value="15.0"/>
+      <mass value="6.0"/>
       <origin xyz="0.0 0 0" rpy=" 0 0 0"/>
       <inertia
@@ -59,5 +59,5 @@
     <pose>0 0 0 0 0 0</pose>
     <inertial>
-      <mass value="2.0"/>
+      <mass value="1"/>
       <origin xyz="0.0 0.0 0.0" rpy="0 1.5707 1.5707"/>
       <inertia
@@ -83,5 +83,5 @@
     <pose>0 0 0 0 0 0</pose>
     <inertial>
-      <mass value="2.0"/>
+      <mass value="1"/>
       <origin xyz="0.0 0.0 0.0" rpy="0 1.5707 1.5707"/>
       <inertia
@@ -185,3 +185,15 @@
     <child link="camera_link_optical"/>
   </joint>
+  <gazebo reference="left_wheel">
+    <material>Gazebo/Black</material>
+  </gazebo>
+  <gazebo reference="right_wheel">
+    <material>Gazebo/Black</material>
+  </gazebo>
+  <gazebo reference="chassis">
+    <material>Gazebo/Red</material>
+  </gazebo>
+  <gazebo reference="camera">
+    <material>Gazebo/Blue</material>
+  </gazebo>
 </robot>
